Commit message: Added visual, collision, inertial and gazebo definitions

File: parsec_description/robot/parsec.urdf (robot description, URDF)
Before this commit: robot parsec, 7 links, 6 joints
Links:
- link base_laser_link: mass None -> 0.001; geometry collision cylinder length=0.08 radius=0.0265; visual cylinder length=0.08 radius=0.0265
- link base_link: mass None -> 15.0; geometry collision cylinder length=0.01 radius=0.21; visual cylinder length=0.01 radius=0.21
- link front_stabilizer_link: mass None -> 0.001; geometry collision box size=0.03 0.03 0.0762; visual box size=0.03 0.03 0.0762
- link left_wheel_link: mass None -> 1.45; geometry collision cylinder length=0.032 radius=0.0762; visual cylinder length=0.032 radius=0.0762
- link mast_link: mass None -> 0.01; geometry collision box size=0.04 0.02 1.65; visual box size=0.04 0.02 1.65
- link rear_stabilizer_link: mass None -> 0.001; geometry collision box size=0.03 0.03 0.0762; visual box size=0.03 0.03 0.0762
- link right_wheel_link: mass None -> 1.45; geometry collision cylinder length=0.032 radius=0.0762; visual cylinder length=0.032 radius=0.0762
Joints:
- joint base_laser_joint: origin xyz=0 0 0.15 -> xyz=0.045 0 -0.68
- joint front_stabilizer_joint: origin xyz=0.195 0 0 -> xyz=0.15 0 0
- joint left_wheel_joint: axis 0 1 0 -> 0 0 1; origin xyz=0 0.195 0 -> xyz=0 0.195 0 rpy=1.5707963268 0 0
- joint mast_joint: origin xyz=0 0 0.005 -> xyz=0 0 0.83
- joint rear_stabilizer_joint: origin xyz=-0.195 0 0 -> xyz=-0.15 0 0
- joint right_wheel_joint: axis 0 1 0 -> 0 0 1; origin xyz=0 -0.195 0 -> xyz=0 -0.195 0 rpy=1.5707963268 0 0

Commit message: Added base_footprint since the base link is a few cm above the ground
Changed configs to account for that.

File: parsec_description/robot/parsec.urdf (robot description, URDF)
Before this commit: robot parsec, 7 links, 6 joints
Links:
- added link base_footprint, mass 0.0001
Joints:
- added joint base_footprint_joint: type fixed, parent base_footprint, child base_link, origin xyz=0 0 0.0762 rpy=0 0 0

Commit message: Renamed base_laser_link to base_laser

File: parsec_description/robot/parsec.urdf (robot description, URDF)
Before this commit: robot parsec, 8 links, 7 joints
Links:
- removed link base_laser_link
- added link base_laser, mass 0.001; collision cylinder length=0.08 radius=0.0265; visual cylinder length=0.08 radius=0.0265
Joints:
- joint base_laser_joint: child base_laser_link -> base_laser

Commit message: Made wheels fixed for now for better visualization in rviz

File: parsec_description/robot/parsec.urdf (robot description, URDF)
Before this commit: robot parsec, 8 links, 7 joints
Joints:
- joint left_wheel_joint: type continuous -> fixed
- joint right_wheel_joint: type continuous -> fixed

Commit message: Added tilting laser to urdf

File: parsec_description/robot/parsec.urdf (robot description, URDF)
Before this commit: robot parsec, 8 links, 7 joints
Links:
- added link tilt_laser, mass 0.001; collision cylinder length=0.08 radius=0.0265; visual cylinder length=0.08 radius=0.0265
- added link tilt_laser_mount, mass 0.001
Joints:
- added joint tilt_laser_joint: type revolute, parent tilt_laser_mount, child tilt_laser, origin xyz=0.0 -0.045 0.035, axis 0 1 0, limit lower=-1.5707963268 upper=1.5707963268 effort=1.0 velocity=10.0
- added joint tilt_laser_mount_joint: type fixed, parent mast_link, child tilt_laser_mount, origin xyz=0.065 0 -0.05

Commit message: Flip the joint axis and change laser orientation slightly
The laser pose sort of fits now. We still need to do a real calibration
however.

File: parsec_description/robot/parsec.urdf (robot description, URDF)
Before this commit: robot parsec, 10 links, 9 joints
Joints:
- joint tilt_laser_joint: origin xyz=0.0 -0.045 0.035 -> xyz=0.0 -0.045 0.035 rpy=0 0.25 0

Commit message: Updating pose of the base laser after using a different mount

File: parsec_description/robot/parsec.urdf (robot description, URDF)
Before this commit: robot parsec, 10 links, 9 joints
Joints:
- joint base_laser_joint: origin xyz=0.045 0 -0.68 -> xyz=0.045 -0.015 -0.68

Commit message: changed orientation and position of tilting laser
The new values are based on finding the ground plane. They should be pretty
accurate now.

File: parsec_description/robot/parsec.urdf (robot description, URDF)
Before this commit: robot parsec, 10 links, 9 joints
Joints:
- joint tilt_laser_joint: origin xyz=0.0 -0.045 0.035 rpy=0 0.25 0 -> xyz=0.0 -0.045 0.033 rpy=0.02 0.215 0

Commit message: Renamed tilt_laser_mount to tilting_laser_mount

File: parsec_description/robot/parsec.urdf (robot description, URDF)
Before this commit: robot parsec, 10 links, 9 joints
Links:
- removed link tilt_laser_mount
- added link tilting_laser_mount, mass 0.001
Joints:
- removed joint tilt_laser_mount_joint
- added joint tilting_laser_mount_joint: type fixed, parent mast_link, child tilting_laser_mount, origin xyz=0.065 0 -0.05
- joint tilt_laser_joint: parent tilt_laser_mount -> tilting_laser_mount

Commit message: Updated URDF

File: parsec_description/robot/parsec.urdf (robot description, URDF)
Before this commit: robot parsec, 10 links, 9 joints
Joints:
- joint tilt_laser_joint: origin xyz=0.0 -0.045 0.033 rpy=0.02 0.215 0 -> xyz=0.0 -0.045 0.033 rpy=0.04 0.00 0.00
- joint tilting_laser_mount_joint: origin xyz=0.065 0 -0.05 -> xyz=0.065 0 -0.12

Commit message: Updated URDF
 * The mast origin is right on top of the base

 * Changed tilt laser position

File: parsec_description/robot/parsec.urdf (robot description, URDF)
Before this commit: robot parsec, 10 links, 9 joints
Joints:
- joint base_laser_joint: origin xyz=0.045 -0.015 -0.68 -> xyz=0.045 -0.015 0.1725
- joint mast_joint: origin xyz=0 0 0.83 -> xyz=0 0 0.0
- joint tilt_laser_joint: origin xyz=0.0 -0.045 0.033 rpy=0.04 0.00 0.00 -> xyz=0.0 -0.045 0.033 rpy=0.02 -0.10 0.00
- joint tilting_laser_mount_joint: origin xyz=0.065 0 -0.12 -> xyz=0.065 0 0.77

Commit message: Fixed position of the base laser

File: parsec_description/robot/parsec.urdf (robot description, URDF)
Before this commit: robot parsec, 10 links, 9 joints
Joints:
- joint base_laser_joint: origin xyz=0.045 -0.015 0.1725 -> xyz=0.06 -0.015 0.18

Commit message: Addressing reviewer comments

File: parsec_description/robot/parsec.urdf (robot description, URDF)
Before this commit: robot parsec, 10 links, 9 joints
Joints:
- joint mast_joint: origin xyz=0 0 0.0 -> xyz=0 0 0

Commit message: Set tilting laser y orientation to zero again
Not sure why this value changed again but zero definitely seems to be the right
value right now.

File: parsec_description/robot/parsec.urdf (robot description, URDF)
Before this commit: robot parsec, 10 links, 9 joints
Joints:
- joint tilt_laser_joint: origin xyz=0.0 -0.045 0.033 rpy=0.02 -0.10 0.00 -> xyz=0.0 -0.045 0.033 rpy=0.02 0.00 0.00

Commit message: Added fixed_angle_laser to urdf

File: parsec_description/robot/parsec.urdf (robot description, URDF)
Before this commit: robot parsec, 10 links, 9 joints
Links:
- added link fixed_angle_laser, mass 0.001; collision cylinder length=0.08 radius=0.0265; visual cylinder length=0.08 radius=0.0265
Joints:
- added joint fixed_angle_laser_joint: type fixed, parent mast_link, child fixed_angle_laser, origin xyz=0.09 0 0.717 rpy=0 0.698 0
