Commit message: Updated parsec urdf to match current configuration with short mast.

File: parsec_description/urdf/parameters.xacro (robot description, xacro)
@@ -3,17 +3,27 @@
        (http://www.ros.org/reps/rep-0103.html).-->
   <!-- Hand measured values. -->
-  <property name="robot_radius" value="0.21" />
+  <property name="base_radius" value="0.21" />
+  <property name="base_height" value="0.01" />
   <property name="wheel_radius" value="0.0762" />
-  <property name="mast_height" value="1.65" />
+  <property name="mast_height" value="0.70" />
+  <!-- Measured from the base. -->
   <property name="base_laser_origin">
-    <origin xyz="0.06 -0.015 0.18" />
+    <origin xyz="0.06 -0.015 0.12" />
   </property>
-  <!-- Calibrated values. See scripts parsec_calibration.-->
-  <property name="tilting_laser_origin">
-    <origin xyz="0.065 -0.045 0.803" rpy="0.02 0.00 0.00" />
+  <!-- Measured from the base -->
+  <property name="servo_axis_origin">
+    <origin xyz="0.065 -0.045 0.625" rpy="0.02 0.00 0.00" />
+  </property>
+  <!-- The distance from the axis of rotation to the origin of the
+       tilting laser sensor. See also
+       parsec_calibration/src/parsec_calibration/servo_calibration_routine.py
+       -->
+  <property name="tilting_laser_offset">
+    <origin xyz="0 0 0.033" />
   </property>
   <property name="fixed_angle_laser_origin">
     <!-- The laser is mounted at an angle of 40 degrees -->
-    <origin xyz="0.09 0 0.717" rpy="0 0.698 0"/>
+    <origin xyz="0.09 0 ${0.851 - base_height / 2 - wheel_radius}"
+            rpy="0 0.698 0"/>
   </property>
 </robot>

File: parsec_description/urdf/parsec.xacro (robot description, xacro)
@@ -46,10 +46,10 @@
       <material name="Black" />
       <geometry>
-        <cylinder radius="${robot_radius}" length="0.01" />
-      </geometry>
-    </visual>
-    <collision>
-      <geometry>
-        <cylinder radius="${robot_radius}" length="0.01" />
+        <cylinder radius="${base_radius}" length="${base_height}" />
+      </geometry>
+    </visual>
+    <collision>
+      <geometry>
+        <cylinder radius="${base_radius}" length="${base_height}" />
       </geometry>
     </collision>
@@ -151,4 +151,5 @@
   </link>
   <laser-link name="base_laser" />
+  <dummy-link name="tilt_laser_base_link" />
   <laser-link name="tilt_laser" />
   <laser-link name="fixed_angle_laser" />
@@ -194,11 +195,16 @@
   <joint name="tilt_laser_joint" type="revolute">
     <parent link="mast_link" />
-    <child link="tilt_laser" />
-    <insert_block name="tilting_laser_origin" />
+    <child link="tilt_laser_base_link" />
+    <insert_block name="servo_axis_origin" />
     <axis xyz="0 1 0" />
     <!-- Using dummy effort and velocity values here. They are not
-         used on the parsec -->
+         used by the controller. -->
     <limit lower="-1.5707963268" upper="1.5707963268"
            effort="1.0" velocity="10.0" />
+  </joint>
+  <joint name="tilt_laser_sensor_joint" type="fixed">
+    <parent link="tilt_laser_base_link" />
+    <child link="tilt_laser" />
+    <insert_block name="tilting_laser_offset" />
   </joint>
   <joint name="fixed_angle_laser_joint" type="fixed">

Commit message: Adjust parameters after calibration.

File: parsec_description/urdf/parameters.xacro (robot description, xacro)
@@ -13,5 +13,5 @@
   <!-- Measured from the base -->
   <property name="servo_axis_origin">
-    <origin xyz="0.065 -0.045 0.625" rpy="0.02 0.00 0.00" />
+    <origin xyz="0.065 -0.045 0.625" rpy="0.00 0.00 0.00" />
   </property>
   <!-- The distance from the axis of rotation to the origin of the

Commit message: Tighten tolerances for tiliting laser.

File: parsec_description/urdf/parameters.xacro (robot description, xacro)
@@ -20,5 +20,5 @@
        -->
   <property name="tilting_laser_offset">
-    <origin xyz="0 0 0.033" />
+    <origin xyz="0 0 0.033" rpy="-0.02 0 0" /> -->
   </property>
   <property name="fixed_angle_laser_origin">

Commit message: Add instructions for brining up the laptop as a base station. Add additional views to rviz config. Tweak URDF params. Tweak floor filter params. Fix gmapping launch file.

File: parsec_description/urdf/parameters.xacro (robot description, xacro)
@@ -9,5 +9,5 @@
   <!-- Measured from the base. -->
   <property name="base_laser_origin">
-    <origin xyz="0.06 -0.015 0.12" />
+    <origin xyz="0.06 -0.015 0.13" />
   </property>
   <!-- Measured from the base -->
@@ -20,5 +20,5 @@
        -->
   <property name="tilting_laser_offset">
-    <origin xyz="0 0 0.033" rpy="-0.02 0 0" /> -->
+    <origin xyz="0 0 0.034" rpy="-0.025 0 0" /> -->
   </property>
   <property name="fixed_angle_laser_origin">

Commit message: Rotated the tilting laser a little bit.

File: parsec_description/urdf/parameters.xacro (robot description, xacro)
@@ -20,5 +20,5 @@
        -->
   <property name="tilting_laser_offset">
-    <origin xyz="0 0 0.034" rpy="-0.025 0 0" /> -->
+    <origin xyz="0 0 0.034" rpy="-0.025 -0.05 0" /> -->
   </property>
   <property name="fixed_angle_laser_origin">

Commit message: Disable the robust relay. It's not necessary in the current configuration and seems to be buggy. Add a note about the sensor origin warning to the move_base_dynamic.launch file. Relax a few floor filter parameters.

File: parsec_description/urdf/parameters.xacro (robot description, xacro)
@@ -9,9 +9,9 @@
   <!-- Measured from the base. -->
   <property name="base_laser_origin">
-    <origin xyz="0.06 -0.015 0.13" />
+    <origin xyz="0.07 -0.015 0.095" />
   </property>
   <!-- Measured from the base -->
   <property name="servo_axis_origin">
-    <origin xyz="0.065 -0.045 0.625" rpy="0.00 0.00 0.00" />
+    <origin xyz="0.085 -0.045 0.38" rpy="0.00 0.00 0.00" />
   </property>
   <!-- The distance from the axis of rotation to the origin of the
@@ -20,10 +20,10 @@
        -->
   <property name="tilting_laser_offset">
-    <origin xyz="0 0 0.034" rpy="-0.025 -0.05 0" /> -->
+    <origin xyz="0 0 0.034" rpy="-0.015 0 0" />
   </property>
   <property name="fixed_angle_laser_origin">
     <!-- The laser is mounted at an angle of 40 degrees -->
-    <origin xyz="0.09 0 ${0.851 - base_height / 2 - wheel_radius}"
-            rpy="-0.04 0.698 0"/>
+    <origin xyz="0.09 0 ${0.8 - base_height / 2 - wheel_radius}"
+            rpy="-0.03 0.698 0"/>
   </property>
 </robot>
